File: pcb/diskohedron4w_hermaphrodit.brd (EAGLE design)
At the start: 88.6 x 57.2 mm, 20 parts, among them X1 87758-1216, X2 87758-1216

Commit message: updated pcb
Parts:
- removed IN1, IN2, OUTR1, OUTR2, U$10, U$9: HERMAPHRODIT4PIN, diskohedron:HERMAPHRODIT4PIN
- added U$11, U$5, U$8: HERMAPHRODITMINI6PIN, diskohedron:HERMAPHRODITMINI6PIN
- added U$12, U$6, U$7: HERMAPHRODIT2PIN, diskohedron:HERMAPHRODIT2PIN
Connections:
- net +24V: now also U$12.P$2, U$6.P$2, U$7.P$2; no longer IN2.P$1, OUTR2.P$4, U$10.P$4
- net CLK+: now also U$8.P$4; no longer IN1.P$4
- net CLK+L: now also U$11.P$1; no longer U$9.P$1
- net CLK+R: now also U$5.P$1; no longer OUTR1.P$1
- net CLK-: now also U$8.P$3; no longer IN1.P$3
- net CLK-L: now also U$11.P$2; no longer U$9.P$2
- net CLK-R: now also U$5.P$2; no longer OUTR1.P$2
- net DATA+: now also U$8.P$2; no longer IN1.P$2
- net DATA-: now also U$8.P$1; no longer IN1.P$1
- net DATAOUT+L: now also U$11.P$3; no longer U$9.P$3
- net DATAOUT+R: now also U$5.P$3; no longer OUTR1.P$3
- net DATAOUT-L: now also U$11.P$4; no longer U$9.P$4
- net DATAOUT-R: now also U$5.P$4; no longer OUTR1.P$4
- net GND: now also U$12.P$1, U$6.P$1, U$7.P$1; no longer IN2.P$2, OUTR2.P$3, U$10.P$3
- net OE+: now also U$8.P$6; no longer IN2.P$4
- net OE+L: now also U$11.P$5; no longer U$10.P$1
- net OE+R: now also U$5.P$5; no longer OUTR2.P$1
- net OE-: no longer IN2.P$3
- net OE-L: now also U$11.P$6; no longer U$10.P$2
- net OE-R: now also U$5.P$6; no longer OUTR2.P$2
Routing:
- net +24V: track 135.5 -> 9.58 mm, vias 3 -> 1
- net GND: track 139.3 -> 126.6 mm
- net CLK+R: track 13.6 -> 6.56 mm
- net OE-L: track 5.93 -> 0.00 mm
- net CLK+L: track 5.93 -> 0.00 mm
- net OE+L: track 5.49 -> 0.00 mm
- net CLK-L: track 5.49 -> 0.00 mm
- net DATAOUT-L: track 5.11 -> 0.00 mm
- net DATAOUT+R: track 11.5 -> 6.66 mm
- net DATA-: track 25.0 -> 20.3 mm
- net DATA+: track 18.5 -> 13.8 mm
- net DATAOUT-R: track 10.2 -> 5.58 mm
- net CLK+: track 94.3 -> 90.9 mm
- net OE+: track 105.4 -> 102.1 mm
- net OE-: track 113.5 -> 110.3 mm
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Other:
- board size 88.6 x 57.2 mm -> 88.5 x 57.3 mm

Commit message: first pcb freeze
Parts:
- added C3, C4: (no value), rcl:C0805
- moved X1 4.29 mm to (67.7, 30.9)
- moved JP1 3.57 mm to (60.0, 13.5)
- moved C2 3.40 mm to (31.6, 6.99)
- moved IC1 2.80 mm to (18.3, 7.31)
- moved U$11 1.59 mm to (21.1, 35.8), turned to 296.6 degrees
- moved U$12 1.54 mm to (17.1, 16.4), turned to 296.6 degrees
- moved X2 1.48 mm to (20.5, 25.9)
- moved U$5 1.40 mm to (66.1, 18.1), turned to 116.6 degrees
- moved U$8 1.25 mm to (64.8, 51.1)
- moved C1 1.05 mm to (75.3, 46.3)
- moved D2 0.94 mm to (36.5, 45.0)
- moved U$1 0.83 mm to (43.5, 27.1), turned to 116.6 degrees
- moved L1 0.82 mm to (44.5, 7.94)
- moved U$6 0.36 mm to (70.2, 37.4), turned to 116.6 degrees
- moved U$7 0.11 mm to (72.7, 46.2)
Connections:
- net +3V3: now also C3.1, C4.1
- net GND: now also C3.2, C4.2, U$2.12
- net OE-: now also U$8.P$5
Routing:
- net +24V: track 9.58 -> 131.2 mm, vias 1 -> 3
- net CLK-: track 97.6 -> 70.7 mm
- net GND: track 126.6 -> 143.7 mm, vias 11 -> 9
- net N$3: track 38.4 -> 23.5 mm, vias 2 -> 4
- net OE+: track 102.1 -> 89.8 mm, vias 3 -> 4
- net DATAOUT+: track 70.9 -> 59.9 mm
- net OE-: track 110.3 -> 102.1 mm
- net +3V3: track 170.2 -> 162.9 mm
- net DATAOUT-: track 65.2 -> 58.1 mm, vias 3 -> 1
- net OE: track 24.8 -> 31.8 mm, vias 1 -> 2
- net OE-L: track 0.00 -> 5.87 mm
- net DATA+: track 13.8 -> 19.3 mm, vias 1 -> 3
- net CLK+L: track 0.00 -> 4.91 mm
- net OE+L: track 0.00 -> 4.79 mm
- net LED3: track 40.1 -> 35.4 mm, vias 1 -> 2
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- removed copper zone on layer 16, net GND
Other:
- board size 88.5 x 57.3 mm -> 94.1 x 58.1 mm
- board text added: "rotation angles: 63.4 26.6"

Commit message: rev. a almost fixed, first gerber-cam process
Parts:
- added U1: SN65LVDS047D, Texas Instruments_By_element14_Batch_1:SOIC127P600X175-16N
- moved D2 20.1 mm to (56.6, 45.0), turned to 90 degrees
- moved JP1 4.59 mm to (59.1, 9.00)
- moved C1 2.11 mm to (73.5, 45.2)
- moved C4 1.71 mm to (43.4, 20.6)
- moved C2 1.68 mm to (30.0, 6.49)
- moved X2 1.49 mm to (21.5, 27.0)
- moved R1 1.39 mm to (45.3, 21.6)
- moved C3 1.21 mm to (55.7, 27.4)
- moved IC1 1.14 mm to (18.0, 8.41)
- moved D1 1.10 mm to (22.4, 17.5)
Connections:
- new net EXTCLK: JP1.4, U1.3
- new net EXTDATA: JP1.3, U1.2
- new net EXTOE: JP1.5, U1.6
- net +3V3: now also U1.1, U1.4
- net CLK: no longer JP1.4
- net CLK+: now also U1.15
- net CLK-: now also U1.16
- net DATA+: now also U1.14
- net DATA-: now also U1.13
- net DATA-IN: no longer JP1.3
- net GND: now also U1.5
- net LED0: now also U$4.7; no longer U$4.1
- net LED3: now also U$4.1; no longer U$4.7
- net OE: no longer JP1.5
- net OE+: now also U1.11
- net OE-: now also U1.12
Routing:
- net +24V: track 131.2 -> 11.3 mm, vias 3 -> 6
- net DATA-: track 19.5 -> 44.6 mm, vias 1 -> 3
- net OE: track 31.8 -> 7.83 mm, vias 2 -> 1
- net +3V3: track 162.9 -> 186.8 mm, vias 4 -> 5
- net N$3: track 23.5 -> 47.1 mm, vias 4 -> 3
- net CLK-: track 70.7 -> 94.2 mm
- net DATA+: track 19.3 -> 40.3 mm
- net OE-: track 102.1 -> 122.5 mm, vias 3 -> 4
- net DATA-IN: track 35.3 -> 15.1 mm
- net CLK: track 38.1 -> 19.2 mm
- net OE+: track 89.8 -> 106.9 mm, vias 4 -> 5
- net CLK+: track 87.6 -> 101.5 mm
- net N$2: track 60.8 -> 51.3 mm, vias 2 -> 1
- net LED3: track 35.4 -> 29.0 mm, vias 2 -> 3
- net LED2: track 23.8 -> 29.2 mm
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- added copper zone on layer 1, net +24V
- added copper zone on layer 16, net +24V
- added copper zone on layer 16, net GND
Other:
- outline, holes or cut-outs redrawn

Commit message: updated gerbers
Parts:
- C3, C4: value (none) -> 100n
- D2: value (none) -> 1n4001
- IC1: value (none) -> LM2596
- JP1: value (none) -> EXTBRD
- moved R1 2.50 mm to (46.0, 24.0), turned to 31.5 degrees
- moved C3 0.86 mm to (55.3, 28.2), turned to 31.5 degrees
- moved C4 0.79 mm to (43.5, 21.3), turned to 31.5 degrees
Routing:
- net GND: track 139.7 -> 111.2 mm, vias 18 -> 16
- net OE-: track 122.5 -> 116.1 mm
- net +24V: track 11.3 -> 8.04 mm
- net +3V3: track 186.8 -> 185.2 mm
- net N$3: track 47.1 -> 46.3 mm
- net CLK+: track 101.5 -> 102.1 mm

Commit message: last commit before changing physical dimension
Parts:
- R1: value (none) -> 220r
- moved JP1 2.34 mm to (59.9, 11.2)
- renumbered IC1 to LM2586, U$1 to STP04, U$11 to OUT-L, U$2 to 4R, U$3 to 1D, U$4 to JST, U$5 to OUT-R, U$8 to IN1, U1 to 4D, X1 to EN-R, X2 to EN-L
Connections:
- net EXTCLK: now also 4D.2, JP1.3; no longer 4D.3, JP1.4
- net EXTDATA: now also 4D.3, JP1.4; no longer 4D.2, JP1.3
Routing:
- net +3V3: track 185.2 -> 180.3 mm
- net GND: track 111.2 -> 113.5 mm
- net EXTOE: track 4.48 -> 3.65 mm
Other:
- board text added: "+24V"
- board text added: "+3V3"
- board text added: "CLK"
- board text added: "DATA"
- board text added: "GND"
- board text added: "INPUT"
- board text added: "L3"
- board text added: "LE"
- board text added: "LED1"
- board text added: "LED2"
- board text added: "OUTPUT-L"
- board text added: "OUTPUT-R"
- board text added: "RED"

Commit message: order for itead 12/05/2014 #100029337
Parts:
- R1: value 220r -> 220R
- moved D1 3.68 mm to (26.1, 17.5)
- moved LM2586 2.40 mm to (20.4, 8.41)
- moved U$7 1.76 mm to (72.6, 44.5)
- moved U$6 1.59 mm to (68.7, 38.0)
- moved C2 1.55 mm to (31.6, 6.79)
- moved EN-R 1.51 mm to (66.8, 29.6)
- moved U$12 1.50 mm to (18.5, 15.9)
- moved EN-L 1.39 mm to (20.9, 25.7)
- moved IN1 1.30 mm to (64.7, 49.8)
- moved OUT-R 1.28 mm to (65.0, 18.6)
- moved OUT-L 1.27 mm to (22.3, 35.3)
- moved JP1 0.70 mm to (59.2, 11.2)
- moved 4D 0.25 mm to (57.8, 25.7)
- moved JST 0.25 mm to (44.9, 47.2)
Routing:
- net GND: track 113.5 -> 94.0 mm
- net +3V3: track 180.3 -> 172.0 mm
- net CLK-: track 94.3 -> 98.2 mm
- net OE+L: track 6.79 -> 3.97 mm
- net +24V: track 8.04 -> 10.5 mm, vias 6 -> 7
- net LED3: track 29.0 -> 31.4 mm
- net OE-L: track 7.74 -> 5.40 mm
- net CLK+R: track 7.87 -> 5.95 mm
- net N$3: track 45.9 -> 47.7 mm
- net DATAOUT+R: track 6.05 -> 4.23 mm
- net DATAOUT-L: track 5.58 -> 3.83 mm
- net DATAOUT-: track 56.2 -> 57.8 mm
- net DATA+: track 40.3 -> 38.8 mm
- net DATA-: track 44.6 -> 43.1 mm
- net N$2: track 51.3 -> 50.0 mm
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Other:
- board size 94.1 x 58.1 mm -> 87.2 x 54.7 mm
- board text added: "05/2014"
- board text added: "DISKO HEDRON"
- board text added: "LED3"
- board text added: "LEDRED"
- board text added: "SAVIC LAMMER SAVICIC"
- board text added: "rev.A"
- board text removed: "L3"
- board text removed: "RED"
