File: pcb/diskohedron4w_revc.brd (EAGLE design)
At the start: 87.2 x 54.7 mm, 61 parts

Commit message: freezing gerber for rev.c, powercone 3d part
Parts:
- TP10, TP9: value TPTP19SQ -> TPTP20SQ; device testpad:TP19SQ -> testpad:TP20SQ
- moved OUT-R1 6.69 mm to (22.6, 4.13)
- moved U$1 6.66 mm to (14.7, 9.45)
- moved TP31 3.16 mm to (42.0, 6.97)
- moved TP32 3.16 mm to (40.1, 6.97)
- moved TP33 3.16 mm to (38.2, 6.97)
- moved TP25 3.15 mm to (42.0, 8.35)
- moved TP26 3.15 mm to (40.1, 8.35)
- moved TP27 3.15 mm to (38.2, 8.35)
- moved LM2586 2.49 mm to (21.6, 9.80)
- moved D1 2.20 mm to (46.2, 6.59)
- moved TP34 1.94 mm to (34.6, 6.84)
- moved TP36 1.94 mm to (30.6, 6.84)
- moved TP35 1.94 mm to (32.5, 6.84)
- moved TP28 1.91 mm to (34.6, 8.22)
- moved TP30 1.91 mm to (30.6, 8.22)
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Routing:
- net N$2: track 50.1 -> 42.9 mm
- net GND: track 30.5 -> 23.5 mm, vias 13 -> 14
- net OE-S: track 3.83 -> 9.35 mm
- net OE+S: track 3.09 -> 7.84 mm
- net DATAOUT+S: track 3.18 -> 6.95 mm
- net CLK-S: track 2.99 -> 6.74 mm
- net +24V: track 22.2 -> 25.8 mm, vias 5 -> 6
- net DATAOUT-S: track 3.47 -> 6.39 mm
- net CLK-: track 110.4 -> 112.7 mm
- net OE+: track 141.8 -> 144.2 mm
- net +3V3: track 192.8 -> 190.7 mm
- net CLK+S: track 3.20 -> 5.36 mm
- net CLK+: track 133.2 -> 135.1 mm, vias 8 -> 7
- net DATAOUT+L: track 6.52 -> 5.63 mm
- net DATAOUT-: track 80.2 -> 81.0 mm
Other:
- board size 87.2 x 54.7 mm -> 87.2 x 55.5 mm
- board text added: "IN-R OUT-R"
- board text added: "OUT-S"
- board text added: "rev.C"
- board text removed: "OUT-R"
- board text removed: "rev.B"
