File: pcb/diskohedron4w_revd.brd (EAGLE design)
At the start: 87.2 x 55.5 mm, 61 parts

Commit message: rev.d and beagle upload scripts
Parts:
- added F1: (no value), adafruit:1812
- moved C2 2.26 mm to (32.5, 6.80)
- moved D1 0.82 mm to (46.0, 5.79)
- moved LM2586 0.40 mm to (21.6, 10.2)
Connections:
- new net IN+24V: C2.+, F1.1, LM2586.1
- net +24V: now also F1.2; no longer C2.+, LM2586.1
Routing:
- net IN+24V: track 0.00 -> 27.0 mm
- net +24V: track 25.8 -> 16.8 mm, vias 6 -> 7
- net N$2: track 42.9 -> 41.0 mm
Other:
- board text added: "10/2014"
- board text added: "rev.D"
- board text removed: "06/2014"
- board text removed: "rev.C"
