File: pcb/diskohedron4w_revd.sch (EAGLE design)
At the start: 61 parts

Commit message: rev.d and beagle upload scripts
Parts:
- added F1: (no value), adafruit:PTCFUSE-1812
Connections:
- new net IN+24V: C2.+, F1.1, LM2586.IN
- net +24V: now also F1.2; no longer C2.+, LM2586.IN
Changed lines of the file:
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@@
 <?xml version="1.0" encoding="utf-8"?>
 <!DOCTYPE eagle SYSTEM "eagle.dtd">
-<eagle version="6.5.0">
+<eagle version="7.0.0">
 <drawing>
 <settings>
@@
 <grid distance="0.1" unitdist="inch" unit="inch" style="lines" multiple="1" display="no" altdistance="0.01" altunitdist="inch" altunit="inch"/>
 <layers>
-<layer number="1" name="Top" color="4" fill="1" visible="no" active="no"/>
-<layer number="16" name="Bottom" color="1" fill="1" visible="no" active="no"/>
-<layer number="17" name="Pads" color="2" fill="1" visible="no" active="no"/>
-<layer number="18" name="Vias" color="2" fill="1" visible="no" active="no"/>
-<layer number="19" name="Unrouted" color="6" fill="1" visible="no" active="no"/>
-<layer number="20" name="Dimension" color="15" fill="1" visible="no" active="no"/>
-<layer number="21" name="tPlace" color="7" fill="1" visible="no" active="no"/>
-<layer number="22" name="bPlace" color="7" fill="1" visible="no" active="no"/>
-<layer number="23" name="tOrigins" color="15" fill="1" visible="no" active="no"/>
-<layer number="24" name="bOrigins" color="15" fill="1" visible="no" active="no"/>
-<layer number="25" name="tNames" color="7" fill="1" visible="no" active="no"/>
-<layer number="26" name="bNames" color="7" fill="1" visible="no" active="no"/>
-<layer number="27" name="tValues" color="7" fill="1" visible="no" active="no"/>
-<layer number="28" name="bValues" color="7" fill="1" visible="no" active="no"/>
+<layer number="1" name="Top" color="4" fill="1" visible="yes" active="no"/>
+<layer number="16" name="Bottom" color="1" fill="1" visible="yes" active="no"/>
+<layer number="17" name="Pads" color="2" fill="1" visible="yes" active="no"/>
+<layer number="18" name="Vias" color="2" fill="1" visible="yes" active="no"/>
+<layer number="19" name="Unrouted" color="6" fill="1" visible="yes" active="no"/>
+<layer number="20" name="Dimension" color="15" fill="1" visible="yes" active="no"/>
+<layer number="21" name="tPlace" color="7" fill="1" visible="yes" active="no"/>
+<layer number="22" name="bPlace" color="7" fill="1" visible="yes" active="no"/>
+<layer number="23" name="tOrigins" color="15" fill="1" visible="yes" active="no"/>
+<layer number="24" name="bOrigins" color="15" fill="1" visible="yes" active="no"/>
+<layer number="25" name="tNames" color="7" fill="1" visible="yes" active="no"/>
+<layer number="26" name="bNames" color="7" fill="1" visible="yes" active="no"/>
+<layer number="27" name="tValues" color="7" fill="1" visible="yes" active="no"/>
+<layer number="28" name="bValues" color="7" fill="1" visible="yes" active="no"/>
 <layer number="29" name="tStop" color="7" fill="3" visible="no" active="no"/>
 <layer number="30" name="bStop" color="7" fill="6" visible="no" active="no"/>
@@
 <layer number="35" name="tGlue" color="7" fill="4" visible="no" active="no"/>
 <layer number="36" name="bGlue" color="7" fill="5" visible="no" active="no"/>
-<layer number="37" name="tTest" color="7" fill="1" visible="no" active="no"/>
-<layer number="38" name="bTest" color="7" fill="1" visible="no" active="no"/>
+<layer number="37" name="tTest" color="7" fill="1" visible="yes" active="no"/>
+<layer number="38" name="bTest" color="7" fill="1" visible="yes" active="no"/>
 <layer number="39" name="tKeepout" color="4" fill="11" visible="no" active="no"/>
 <layer number="40" name="bKeepout" color="1" fill="11" visible="no" active="no"/>
@@
 <layer number="44" name="Drills" color="7" fill="1" visible="no" active="no"/>
 <layer number="45" name="Holes" color="7" fill="1" visible="no" active="no"/>
-<layer number="46" name="Milling" color="3" fill="1" visible="no" active="no"/>
-<layer number="47" name="Measures" color="7" fill="1" visible="no" active="no"/>
-<layer number="48" name="Document" color="7" fill="1" visible="no" active="no"/>
-<layer number="49" name="Reference" color="7" fill="1" visible="no" active="no"/>
-<layer number="50" name="dxf" color="7" fill="1" visible="no" active="no"/>
-<layer number="51" name="tDocu" color="7" fill="1" visible="no" active="no"/>
-<layer number="52" name="bDocu" color="7" fill="1" visible="no" active="no"/>
-<layer number="53" name="tGND_GNDA" color="7" fill="1" visible="no" active="no"/>
-<layer number="54" name="bGND_GNDA" color="7" fill="1" visible="no" active="no"/>
-<layer number="56" name="wert" color="7" fill="1" visible="no" active="no"/>
-<layer number="57" name="tCAD" color="7" fill="1" visible="no" active="no"/>
+<layer number="46" name="Milling" color="3" fill="1" visible="yes" active="no"/>
+<layer number="47" name="Measures" color="7" fill="1" visible="yes" active="no"/>
+<layer number="48" name="Document" color="7" fill="1" visible="yes" active="no"/>
+<layer number="49" name="Reference" color="7" fill="1" visible="yes" active="no"/>
+<layer number="50" name="dxf" color="7" fill="1" visible="yes" active="no"/>
+<layer number="51" name="tDocu" color="7" fill="1" visible="yes" active="no"/>
+<layer number="52" name="bDocu" color="7" fill="1" visible="yes" active="no"/>
+<layer number="53" name="tGND_GNDA" color="7" fill="1" visible="yes" active="no"/>
+<layer number="54" name="bGND_GNDA" color="7" fill="1" visible="yes" active="no"/>
+<layer number="56" name="wert" color="7" fill="1" visible="yes" active="no"/>
+<layer number="57" name="tCAD" color="7" fill="1" visible="yes" active="no"/>
 <layer number="91" name="Nets" color="2" fill="1" visible="yes" active="yes"/>
 <layer number="92" name="Busses" color="1" fill="1" visible="yes" active="yes"/>
@@
 <part name="TP39" library="testpad" deviceset="TP" device="TP09SQ" value="TPTP09SQ"/>
 <part name="TP40" library="testpad" deviceset="TP" device="TP09SQ" value="TPTP09SQ"/>
+<part name="F1" library="adafruit" deviceset="PTCFUSE" device="-1812"/>
 </parts>
 <sheets>
@@
 <attribute name="TP_SIGNAL_NAME" x="39.37" y="31.75" size="1.778" layer="97" rot="R270"/>
 </instance>
+<instance part="F1" gate="G$1" x="44.45" y="123.19"/>
 </instances>
 <busses>
@@
 <net name="+24V" class="0">
 <segment>
-<pinref part="C2" gate="G$1" pin="+"/>
-<label x="45.72" y="223.52" size="1.778" layer="95"/>
-<pinref part="LM2586" gate="G$1" pin="IN"/>
-<wire x1="53.34" y1="220.98" x2="35.56" y2="220.98" width="0.1524" layer="91"/>
-<label x="27.94" y="218.44" size="1.778" layer="95"/>
-<wire x1="35.56" y1="215.9" x2="35.56" y2="220.98" width="0.1524" layer="91"/>
-</segment>
-<segment>
 <pinref part="U$7" gate="G$1" pin="P$2"/>
-<wire x1="29.21" y1="125.73" x2="57.15" y2="125.73" width="0.1524" layer="91"/>
-<label x="29.21" y="125.73" size="1.778" layer="95"/>
+<wire x1="57.15" y1="125.73" x2="49.53" y2="125.73" width="0.1524" layer="91"/>
+<pinref part="F1" gate="G$1" pin="2"/>
+<label x="50.8" y="127" size="1.778" layer="95"/>
+</segment>
+<segment>
+<pinref part="U$12" gate="G$1" pin="P$1"/>
+<wire x1="115.57" y1="133.35" x2="86.36" y2="133.35" width="0.1524" layer="91"/>
+<label x="86.36" y="133.35" size="1.778" layer="95"/>
+</segment>
+<segment>
+<wire x1="57.15" y1="82.55" x2="29.21" y2="82.55" width="0.1524" layer="91"/>
+<label x="29.21" y="82.55" size="1.778" layer="95"/>
+<pinref part="U$1" gate="G$1" pin="P$2"/>
 </segment>
 <segment>
@@
 <label x="87.63" y="90.17" size="1.778" layer="95"/>
 <pinref part="U$6" gate="G$1" pin="P$1"/>
-</segment>
-<segment>
-<pinref part="U$12" gate="G$1" pin="P$1"/>
-<wire x1="115.57" y1="133.35" x2="86.36" y2="133.35" width="0.1524" layer="91"/>
-<label x="86.36" y="133.35" size="1.778" layer="95"/>
-</segment>
-<segment>
-<wire x1="57.15" y1="82.55" x2="29.21" y2="82.55" width="0.1524" layer="91"/>
-<label x="29.21" y="82.55" size="1.778" layer="95"/>
-<pinref part="U$1" gate="G$1" pin="P$2"/>
 </segment>
 </net>
@@
 </segment>
 </net>
+<net name="IN+24V" class="0">
+<segment>
+<pinref part="F1" gate="G$1" pin="1"/>
+<wire x1="39.37" y1="125.73" x2="29.21" y2="125.73" width="0.1524" layer="91"/>
+<label x="27.94" y="127" size="1.778" layer="95"/>
+</segment>
+<segment>
+<pinref part="C2" gate="G$1" pin="+"/>
+<label x="45.72" y="223.52" size="1.778" layer="95"/>
+<pinref part="LM2586" gate="G$1" pin="IN"/>
+<wire x1="53.34" y1="220.98" x2="35.56" y2="220.98" width="0.1524" layer="91"/>
+<label x="27.94" y="218.44" size="1.778" layer="95"/>
+<wire x1="35.56" y1="215.9" x2="35.56" y2="220.98" width="0.1524" layer="91"/>
+</segment>
+</net>
